File: electronics/v1/flute.brd (EAGLE design)
At the start: 32 x 250 mm, 47 parts, among them P1 PRESSURE_SENSOR, Q1 BC550C, Q2 BC550C

Commit message: v1.01
Parts:
- added U$10, U$11, U$12, U$13, U$15, U$4, U$5, U$6, U$7, U$8: (no value), rhoban:M25_HOLE
- U$1, U$2: device SparkFun-Electromechanical:STAND-OFF -> rhoban:M25_HOLE
- moved U$1 48.3 mm to (2.30, 51.4)
- moved U$14 24.0 mm to (12.0, 205.0), turned to 0 degrees
- moved R19 20.6 mm to (10.1, 13.9), turned to 180 degrees
- moved C1 18.3 mm to (9.62, 31.2)
- moved R20 18.3 mm to (9.62, 28.1)
- moved SPEAKER 17.3 mm to (14.3, 31.3), turned to 180 degrees
- moved R21 17.1 mm to (11.0, 33.7)
- moved JMP 14.3 mm to (25.8, 210.8)
- moved R23 14.2 mm to (11.3, 47.7)
- moved PWR 11.8 mm to (25.8, 216.9)
- moved R22 10.5 mm to (9.72, 47.7), turned to 90 degrees
- moved R2 7.55 mm to (15.1, 160.9), turned to 90 degrees
- moved U$9 7.07 mm to (12.0, 228.0)
- moved Q2 6.32 mm to (19.0, 162.1)
- moved AMP 4.14 mm to (13.3, 40.7), flipped to the bottom
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Routing:
- net GND: track 424.3 -> 0.00 mm, vias 3 -> 0
- net VCC: track 285.3 -> 0.00 mm, vias 3 -> 0
- net PRESSURE: track 229.6 -> 0.00 mm, vias 1 -> 0
- net VIN: track 224.2 -> 0.00 mm, vias 3 -> 0
- net HOLE8: track 177.2 -> 0.00 mm
- net HOLE1: track 159.6 -> 0.00 mm, vias 1 -> 0
- net HOLES_GND2: track 147.4 -> 0.00 mm
- net HOLE2: track 145.0 -> 0.00 mm, vias 1 -> 0
- net HOLE3: track 136.5 -> 0.00 mm, vias 1 -> 0
- net HOLES_EN: track 131.2 -> 0.00 mm, vias 2 -> 0
- net HOLES_GND1: track 121.7 -> 0.00 mm
- net HOLE4: track 105.9 -> 0.00 mm, vias 1 -> 0
- net HOLE5: track 96.7 -> 0.00 mm
- net HOLE6: track 69.3 -> 0.00 mm, vias 1 -> 0
- net HOLE7: track 51.4 -> 0.00 mm
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Other:
- board size 32 x 250 mm -> 27 x 250 mm

Commit message: Routed V1 (to be checked)
Parts:
- added U$16: SWITCHKCD11, rhoban:KCD11
- added U$18, U$19, U$20, U$21, U$22, U$23: SWITCH6X6X10, rhoban:SWITCH_6X6X10
- moved PWR 135.6 mm to (25.4, 81.3)
- moved JMP 122.9 mm to (25.4, 87.9)
- moved Q2 66.7 mm to (20.4, 95.4)
- moved R2 66.6 mm to (16.5, 94.3)
- moved Q1 66.4 mm to (9.01, 95.3)
- moved R1 66.4 mm to (13.5, 94.4)
- moved U$9 3.20 mm to (14.5, 226.0)
- moved U$11 3.00 mm to (27.7, 198.7)
- moved U$13 3.00 mm to (27.7, 247.8)
- moved U$14 3.00 mm to (15.0, 205.0)
- moved U$2 3.00 mm to (27.7, 2.30)
- moved U$4 3.00 mm to (27.7, 51.4)
- moved U$6 3.00 mm to (27.7, 100.5)
- moved U$8 3.00 mm to (27.7, 149.6)
- moved U$3 2.24 mm to (14.0, 214.2)
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Connections:
- removed net SD_CS: MAPLE.X20
- removed net SD_MISO: MAPLE.X18
- removed net SD_MOSI: MAPLE.X17
- removed net SD_SCK: MAPLE.X19
- new net BUT1: MAPLE.X15, U$18.B1, U$18.B2
- new net BUT2: MAPLE.X16, U$19.B1, U$19.B2
- new net BUT3: MAPLE.X17, U$20.B1, U$20.B2
- new net BUT4: MAPLE.X18, U$21.B1, U$21.B2
- new net BUT5: MAPLE.X19, U$22.B1, U$22.B2
- new net BUT6: MAPLE.X20, U$23.B1, U$23.B2
- new net VIN_BAT: PWR.1, U$16.A1, U$16.A2
- net GND: now also U$18.A1, U$18.A2, U$19.A1, U$19.A2, U$20.A1, U$20.A2, U$21.A1, U$21.A2, U$22.A1, U$22.A2, U$23.A1, U$23.A2
- net VIN: now also U$16.B1, U$16.B2; no longer PWR.1
Routing:
- net GND: track 0.00 -> 372.0 mm, vias 0 -> 1
- net VCC: track 0.00 -> 319.2 mm, vias 0 -> 6
- net PRESSURE: track 0.00 -> 250.3 mm, vias 0 -> 3
- net BUT1: track 0.00 -> 217.5 mm, vias 0 -> 5
- net VIN: track 0.00 -> 191.3 mm, vias 0 -> 3
- net HOLE8: track 0.00 -> 180.4 mm, vias 0 -> 4
- net HOLE1: track 0.00 -> 175.1 mm, vias 0 -> 3
- net BUT2: track 0.00 -> 171.9 mm, vias 0 -> 3
- net BUT3: track 0.00 -> 171.7 mm, vias 0 -> 4
- net BUT5: track 0.00 -> 171.0 mm, vias 0 -> 4
- net BUT4: track 0.00 -> 161.6 mm, vias 0 -> 6
- net HOLE3: track 0.00 -> 156.4 mm, vias 0 -> 4
- net HOLE2: track 0.00 -> 151.0 mm, vias 0 -> 2
- net BUT6: track 0.00 -> 147.7 mm, vias 0 -> 1
- net HOLES_GND2: track 0.00 -> 133.0 mm
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Other:
- board size 27 x 250 mm -> 30 x 250 mm

Commit message: up
Parts:
- added U$24: HC05, rhoban:HC-05
- U$17: value RHOBAN_MCP4822 -> MCP4822
- moved MAPLE 14.2 mm to (8.43, 1.33), flipped to the top
- moved U$11 2.00 mm to (29.7, 198.7)
- moved U$13 2.00 mm to (29.7, 247.8)
- moved U$2 2.00 mm to (29.7, 2.30)
- moved U$4 2.00 mm to (29.7, 51.4)
- moved U$6 2.00 mm to (29.7, 100.5)
- moved U$8 2.00 mm to (29.7, 149.6)
- moved SPEAKER 1.29 mm to (17.1, 31.3), flipped to the bottom
- moved P1 1.12 mm to (21.8, 244.7)
- moved R21 1.10 mm to (13.6, 33.8), flipped to the bottom, turned to 0 degrees
- moved AMP 1.00 mm to (15.8, 40.7)
- moved JACK 1.00 mm to (16.0, 5.85)
- moved JMP 1.00 mm to (26.4, 87.9)
- moved OS1 1.00 mm to (15.9, 194.8)
- moved OS2 1.00 mm to (15.9, 172.8)
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Connections:
- removed net N$16: C1.1, R20.2
- new net KEY: MAPLE.X22, U$24.KEY
- new net N$12: C1.2, R20.1
- new net RX1: MAPLE.X25, U$24.TX
- new net TX1: MAPLE.X26, U$24.RX
- net 33: now also U$24.3.3
- net GND: now also U$24.GND; no longer R22.2
- net N$18: now also R20.2; no longer C1.2
- net N$20: now also C1.1; no longer R20.1
- net VIN: now also R22.2
Routing:
- net 33: track 0.00 -> 167.9 mm, vias 0 -> 2
- net KEY: track 0.00 -> 126.9 mm, vias 0 -> 4
- net TX1: track 0.00 -> 121.8 mm, vias 0 -> 6
- net RX1: track 0.00 -> 121.3 mm, vias 0 -> 9
- net VIN: track 191.3 -> 269.2 mm, vias 3 -> 6
- net GND: track 372.0 -> 436.1 mm, vias 1 -> 8
- net HOLE6: track 90.7 -> 130.2 mm, vias 3 -> 2
- net VCC: track 319.2 -> 289.5 mm, vias 6 -> 3
- net PRESSURE: track 250.3 -> 225.7 mm, vias 3 -> 4
- net BUT4: track 161.6 -> 182.6 mm, vias 6 -> 0
- net HOLE3: track 156.4 -> 137.1 mm, vias 4 -> 1
- net DAC_SCK: track 50.6 -> 34.3 mm, vias 1 -> 2
- net BUT2: track 171.9 -> 188.1 mm
- net N$14: track 9.96 -> 22.5 mm, vias 1 -> 0
- net HOLE5: track 95.0 -> 83.4 mm, vias 6 -> 2
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- added copper zone on layer 1, net GND
- added copper zone on layer 16, net GND
Other:
- board size 30 x 250 mm -> 32 x 250 mm

Commit message: Fixes
Parts:
- R1, R2: value 10k -> 1k
Connections:
- removed net N$6: JACK.1
- net GND: now also JACK.1
Changed lines of the file:
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@@
 <element name="Q1" library="transistor-npn" package="TO92-EBC" value="BC550C" x="10.005178125" y="95.29793125" rot="R90"/>
 <element name="Q2" library="transistor-npn" package="TO92-EBC" value="BC550C" x="21.413728125" y="95.38474375" rot="R270"/>
-<element name="R1" library="SparkFun-Passives" package="0805" value="10k" x="14.52214375" y="94.398053125" rot="R90"/>
-<element name="R2" library="SparkFun-Passives" package="0805" value="10k" x="17.527284375" y="94.34596875" rot="R90"/>
+<element name="R1" library="SparkFun-Passives" package="0805" value="1k" x="14.52214375" y="94.398053125" rot="R90"/>
+<element name="R2" library="SparkFun-Passives" package="0805" value="1k" x="17.527284375" y="94.34596875" rot="R90"/>
 <element name="U$17" library="rhoban" package="DIL08" value="MCP4822" x="15.967271875" y="20.62776875" rot="MR270"/>
 <element name="P1" library="rhoban" package="MPXV5050GP" value="PRESSURE_SENSOR" x="21.7795375" y="244.67186875" rot="R180"/>
@@
 <vertex x="-36.6" y="210.6"/>
 </polygon>
+<contactref element="JACK" pad="1"/>
+<wire x1="16.03473125" y1="5.8522625" x2="23.669709375" y2="3.871515625" width="0" layer="19" extent="1-1"/>
 </signal>
 <signal name="VCC">
@@
 <wire x1="19.6" y1="44.6" x2="19.63756875" y2="44.52280625" width="0.3048" layer="16"/>
 </signal>
-<signal name="N$6">
-<contactref element="JACK" pad="1"/>
-</signal>
 <signal name="N$8">

Commit message: Fixes
Parts:
- removed U$3: AP1117E50G-13, rhoban:SOT223
- added U$25: MCP1703T-5002EDB, rhoban:SOT223
Connections:
- net GND: now also U$25.2; no longer U$3.1
- net VCC: now also U$25.3; no longer R13.1, R14.1, R15.1, R16.1, R17.1, R18.1, R4.1, R6.2, U$3.2
- net VIN: now also R13.1, R14.1, R15.1, R16.1, R17.1, R18.1, R4.1, R6.2, U$25.1; no longer U$3.3
Routing:
- net GND: track 436.1 -> 0.00 mm, vias 8 -> 0
- net VCC: track 289.5 -> 0.00 mm, vias 3 -> 0
- net VIN: track 269.2 -> 0.00 mm, vias 6 -> 0
- net PRESSURE: track 225.7 -> 0.00 mm, vias 4 -> 0
- net BUT1: track 209.2 -> 0.00 mm, vias 5 -> 0
- net BUT2: track 188.1 -> 0.00 mm, vias 3 -> 0
- net BUT4: track 182.6 -> 0.00 mm
- net HOLE8: track 175.8 -> 0.00 mm, vias 1 -> 0
- net BUT5: track 174.9 -> 0.00 mm, vias 3 -> 0
- net HOLE1: track 169.1 -> 0.00 mm, vias 4 -> 0
- net 33: track 167.9 -> 0.00 mm, vias 2 -> 0
- net BUT3: track 166.3 -> 0.00 mm, vias 4 -> 0
- net BUT6: track 156.2 -> 0.00 mm, vias 5 -> 0
- net HOLE2: track 150.1 -> 0.00 mm
- net HOLE3: track 137.1 -> 0.00 mm, vias 1 -> 0
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- removed copper zone on layer 1, net GND
- removed copper zone on layer 16, net GND
