File: electronics/v1.1/flute.brd (EAGLE design)
At the start: 32 x 250 mm, 65 parts, among them P1 PRESSURE_SENSOR, Q1 BC550C, Q2 BC550C

Commit message: elec
Parts:
- added IC1: TP4056, TP4056:SOP-8
- added R24, R25, R28: 2K, SparkFun-Passives:0805
- added R26, R27: 270, SparkFun-Passives:0805
- added U$15, U$26: LED_3MM, rhoban:LED3MM
- added U$27: NPN_BC817,215, rhoban:SOT-23
- moved U$25 141.9 mm to (9.40, 72.2)
- moved U$18 51.0 mm to (24.5, 219.2)
- moved U$19 51.0 mm to (13.4, 219.2)
- moved U$20 50.0 mm to (24.5, 212.0)
- moved U$21 50.0 mm to (13.4, 212.0)
- moved U$22 49.0 mm to (24.5, 204.7)
- moved U$23 49.0 mm to (13.4, 204.7)
- moved U$14 26.1 mm to (21.5, 230.5)
- moved U$9 6.02 mm to (11.5, 230.5), turned to 0 degrees
- moved U$24 0.50 mm to (21.0, 138.0)
Connections:
- new net 3.3: U$25.3
- new net CHARGE_EN: IC1.8, R25.1, U$27.3
- new net N$16: R26.2, U$15.A
- new net N$21: IC1.2, R24.2
- new net N$22: R28.1, U$27.1
- new net N$24: IC1.7, U$15.K
- new net N$25: IC1.6, U$26.K
- new net N$6: R27.2, U$26.A
- net GND: now also IC1.1, IC1.3, R24.1, U$27.2
- net VCC: now also IC1.4, R25.2, R26.1, R27.1; no longer U$25.3
- net VIN: now also R28.2
- net VIN_BAT: now also IC1.5

Commit message: elec v1.1 (wip)
Parts:
- removed JMP: CONNEC_1X02BASIC, rhoban:CONNEC_1X02
- removed Q1, Q2: BC550C, transistor-npn:TO92-EBC
- added SU-5V: STEPUP-5V, rhoban:STEPUP-5V
- added U$28, U$29: NPN_BC817,215, rhoban:SOT-23
- moved U$25 27.5 mm to (30.4, 90.0), flipped to the bottom
- moved R2 11.6 mm to (7.40, 88.8), turned to 180 degrees
- moved R28 11.3 mm to (33.5, 63.0), turned to 90 degrees
- moved R24 10.4 mm to (31.2, 63.0), turned to 270 degrees
- moved U$27 9.38 mm to (32.5, 59.2)
- moved R25 9.09 mm to (32.5, 56.2)
- moved PWR 7.50 mm to (32.9, 77.5)
- moved R1 7.30 mm to (7.35, 93.0), turned to 180 degrees
- moved R26 4.28 mm to (7.25, 64.2)
- moved R27 4.28 mm to (7.25, 59.5), turned to 180 degrees
- moved U$26 4.03 mm to (3.00, 59.5)
- moved U$15 4.01 mm to (3.00, 64.5)
- moved SPEAKER 3.38 mm to (19.9, 29.4), turned to 0 degrees
- moved U$11 3.00 mm to (32.7, 198.7)
- moved U$13 3.00 mm to (32.7, 247.8)
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Connections:
- new net USB+: IC1.4, MAPLE.VIN, R25.2
- net GND: now also SU-5V.IN-, SU-5V.OUT-, U$28.2, U$29.2; no longer Q1.E, Q2.E
- net HOLES_GND1: now also U$28.3; no longer Q1.C
- net HOLES_GND2: now also U$29.3; no longer Q2.C
- net N$3: now also U$28.1; no longer Q1.B
- net N$4: now also U$29.1; no longer Q2.B
- net VCC: now also AMP.5, R22.2, SU-5V.OUT+; no longer IC1.4, JMP.2, MAPLE.VIN, R25.2
- net VIN: now also MAPLE.X21, SU-5V.IN+; no longer AMP.5, JMP.1, R22.2
Routing:
- net GND: track 0.00 -> 504.4 mm, vias 0 -> 16
- net VIN: track 0.00 -> 361.0 mm, vias 0 -> 13
- net VCC: track 0.00 -> 306.0 mm, vias 0 -> 12
- net BUT2: track 0.00 -> 243.9 mm, vias 0 -> 6
- net PRESSURE: track 0.00 -> 227.6 mm, vias 0 -> 8
- net BUT4: track 0.00 -> 227.5 mm, vias 0 -> 6
- net BUT1: track 0.00 -> 223.5 mm, vias 0 -> 3
- net BUT3: track 0.00 -> 212.7 mm, vias 0 -> 2
- net HOLES_GND2: track 0.00 -> 211.6 mm, vias 0 -> 3
- net BUT6: track 0.00 -> 205.0 mm, vias 0 -> 5
- net BUT5: track 0.00 -> 200.3 mm, vias 0 -> 4
- net HOLE8: track 0.00 -> 169.3 mm, vias 0 -> 4
- net HOLE1: track 0.00 -> 165.2 mm, vias 0 -> 2
- net HOLES_GND1: track 0.00 -> 148.2 mm, vias 0 -> 3
- net HOLE2: track 0.00 -> 143.8 mm, vias 0 -> 2
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Other:
- board size 32 x 250 mm -> 35 x 250 mm

Commit message: v1.1
Parts:
- added C2, C3: 10uF, SparkFun-Passives:0805
- added R29: 0.4, SparkFun-Passives:0805
- added U$30: 47uF, rhoban:PANASONIC_D
- moved PWR 1.77 mm to (32.7, 79.3)
- moved U$15 1.00 mm to (4.00, 64.5)
- moved U$26 1.00 mm to (4.00, 59.5)
- moved SU-5V 0.56 mm to (23.8, 98.5)
- turned R26 to 270 degrees
- turned R27 to 90 degrees
Connections:
- removed net 3.3: U$25.3
- removed net HOLES_EN: MAPLE.X2, R1.1, R2.1
- new net HOLES_EN1: MAPLE.X12, R1.1
- new net HOLES_EN2: MAPLE.X13, R2.1
- new net N$23: C2.2, IC1.4, R29.2
- net 33: now also U$25.3, U$30.+
- net GND: now also C2.1, C3.1, U$30.-
- net USB+: no longer IC1.4
- net VCC: now also R29.1; no longer R10.2, R11.2, R12.2, R3.1, R5.1, R7.2, R8.2, R9.2
- net VIN: now also R10.2, R11.2, R12.2, R3.1, R5.1, R7.2, R8.2, R9.2
- net VIN_BAT: now also C3.2
Routing:
- net HOLES_EN1: track 0.00 -> 90.2 mm, vias 0 -> 6
- net HOLES_EN2: track 0.00 -> 80.3 mm, vias 0 -> 2
- net USB+: track 39.1 -> 116.3 mm, vias 5 -> 4
- net HOLES_GND2: track 211.6 -> 145.1 mm, vias 3 -> 6
- net HOLE6: track 135.1 -> 70.6 mm, vias 2 -> 3
- net TX1: track 112.0 -> 168.5 mm, vias 3 -> 6
- net HOLES_EN: track 53.0 -> 0.00 mm, vias 3 -> 0
- net VIN: track 361.0 -> 316.6 mm, vias 13 -> 6
- net DAC_SCK: track 86.6 -> 45.3 mm, vias 2 -> 0
- net N$25: track 68.5 -> 30.2 mm, vias 4 -> 1
- net BUT1: track 223.5 -> 258.7 mm, vias 3 -> 2
- net PRESSURE: track 227.6 -> 261.7 mm, vias 8 -> 6
- net VCC: track 306.0 -> 275.1 mm, vias 12 -> 10
- net KEY: track 123.6 -> 143.2 mm, vias 3 -> 4
- net DAC_SDI: track 50.6 -> 32.3 mm, vias 2 -> 0
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- added copper zone on layer 1, net GND
- added copper zone on layer 16, net GND
