File: electronics/v1.1/flute.sch (EAGLE design)
At the start: 53 parts, among them P1 PRESSURE_SENSOR, Q1 BC550C, Q2 BC550C

Commit message: elec
Parts:
- added IC1: TP4056, TP4056:TP4056
- added R24, R25, R28: 2K, SparkFun-Passives:RESISTOR0805-RES
- added R26, R27: 270, SparkFun-Passives:RESISTOR0805-RES
- added U$15, U$26: LED_3MM, rhoban:LED_3MM
- added U$27: NPN_BC817,215, rhoban:NPN_BC817,215
Connections:
- new net 3.3: U$25.OUT
- new net CHARGE_EN: IC1.CE, R25.1, U$27.C
- new net N$16: R26.2, U$15.A
- new net N$21: IC1.PROG, R24.2
- new net N$22: R28.1, U$27.B
- new net N$24: IC1.CHRG, U$15.C
- new net N$25: IC1.STDBY, U$26.C
- new net N$6: R27.2, U$26.A
- net GND: now also IC1.GND, IC1.TEMP, R24.1, U$27.E
- net VCC: now also IC1.VCC, R25.2, R26.1, R27.1; no longer U$25.OUT
- net VIN: now also R28.2
- net VIN_BAT: now also IC1.BAT
Changed lines of the file:
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@@
 <part name="U$24" library="rhoban" deviceset="HC05" device=""/>
 <part name="U$25" library="rhoban" deviceset="MCP1703T-5002EDB" device=""/>
+<part name="IC1" library="TP4056" deviceset="TP4056" device=""/>
+<part name="R24" library="SparkFun-Passives" deviceset="RESISTOR" device="0805-RES" value="2K"/>
+<part name="R25" library="SparkFun-Passives" deviceset="RESISTOR" device="0805-RES" value="2K"/>
+<part name="U$15" library="rhoban" deviceset="LED_3MM" device=""/>
+<part name="U$26" library="rhoban" deviceset="LED_3MM" device=""/>
+<part name="R26" library="SparkFun-Passives" deviceset="RESISTOR" device="0805-RES" value="270"/>
+<part name="R27" library="SparkFun-Passives" deviceset="RESISTOR" device="0805-RES" value="270"/>
+<part name="U$27" library="rhoban" deviceset="NPN" device="_BC817,215"/>
+<part name="R28" library="SparkFun-Passives" deviceset="RESISTOR" device="0805-RES" value="2K"/>
 </parts>
 <sheets>
@@
 <instance part="U$24" gate="G$1" x="33.02" y="27.94"/>
 <instance part="U$25" gate="G$1" x="81.28" y="-101.6"/>
+<instance part="IC1" gate="G$1" x="104.14" y="-119.38"/>
+<instance part="R24" gate="G$1" x="83.82" y="-124.46"/>
+<instance part="R25" gate="G$1" x="139.7" y="-116.84" rot="R90"/>
+<instance part="U$15" gate="G$1" x="134.62" y="-124.46" rot="R270"/>
+<instance part="U$26" gate="G$1" x="134.62" y="-127" rot="R270"/>
+<instance part="R26" gate="G$1" x="144.78" y="-124.46" rot="R180"/>
+<instance part="R27" gate="G$1" x="144.78" y="-127" rot="R180"/>
+<instance part="U$27" gate="G$1" x="187.96" y="-127"/>
+<instance part="R28" gate="G$1" x="177.8" y="-127" rot="R180"/>
 </instances>
 <busses>
@@
 <label x="73.66" y="-106.68" size="1.778" layer="95"/>
 </segment>
+<segment>
+<pinref part="IC1" gate="G$1" pin="GND"/>
+<wire x1="99.06" y1="-127" x2="96.52" y2="-127" width="0.1524" layer="91"/>
+<label x="88.9" y="-127" size="1.778" layer="95"/>
+</segment>
+<segment>
+<pinref part="IC1" gate="G$1" pin="TEMP"/>
+<wire x1="99.06" y1="-121.92" x2="96.52" y2="-121.92" width="0.1524" layer="91"/>
+<label x="88.9" y="-121.92" size="1.778" layer="95"/>
+</segment>
+<segment>
+<pinref part="R24" gate="G$1" pin="1"/>
+<wire x1="78.74" y1="-124.46" x2="76.2" y2="-124.46" width="0.1524" layer="91"/>
+<label x="71.12" y="-124.46" size="1.778" layer="95"/>
+</segment>
+<segment>
+<pinref part="U$27" gate="G$1" pin="E"/>
+<wire x1="190.5" y1="-132.08" x2="190.5" y2="-134.62" width="0.1524" layer="91"/>
+<label x="190.5" y="-137.16" size="1.778" layer="95"/>
+</segment>
 </net>
 <net name="VCC" class="0">
@@
 </segment>
 <segment>
-<pinref part="U$25" gate="G$1" pin="OUT"/>
-<wire x1="88.9" y1="-93.98" x2="91.44" y2="-93.98" width="0.1524" layer="91"/>
-<label x="91.44" y="-93.98" size="1.778" layer="95"/>
+<pinref part="IC1" gate="G$1" pin="VCC"/>
+<wire x1="99.06" y1="-129.54" x2="96.52" y2="-129.54" width="0.1524" layer="91"/>
+<label x="88.9" y="-129.54" size="1.778" layer="95"/>
+</segment>
+<segment>
+<pinref part="R25" gate="G$1" pin="2"/>
+<wire x1="139.7" y1="-111.76" x2="139.7" y2="-109.22" width="0.1524" layer="91"/>
+<label x="139.7" y="-109.22" size="1.778" layer="95"/>
+</segment>
+<segment>
+<pinref part="R26" gate="G$1" pin="1"/>
+<wire x1="149.86" y1="-124.46" x2="152.4" y2="-124.46" width="0.1524" layer="91"/>
+<label x="152.4" y="-124.46" size="1.778" layer="95"/>
+</segment>
+<segment>
+<pinref part="R27" gate="G$1" pin="1"/>
+<wire x1="149.86" y1="-127" x2="152.4" y2="-127" width="0.1524" layer="91"/>
+<label x="152.4" y="-127" size="1.778" layer="95"/>
 </segment>
 </net>
@@
 <wire x1="58.42" y1="-93.98" x2="55.88" y2="-93.98" width="0.1524" layer="91"/>
 <label x="50.8" y="-93.98" size="1.778" layer="95"/>
+</segment>
+<segment>
+<wire x1="172.72" y1="-127" x2="170.18" y2="-127" width="0.1524" layer="91"/>
+<label x="167.64" y="-127" size="1.778" layer="95"/>
+<pinref part="R28" gate="G$1" pin="2"/>
 </segment>
 </net>
@@
 <label x="68.58" y="-55.88" size="1.778" layer="95"/>
 </segment>
+<segment>
+<pinref part="IC1" gate="G$1" pin="BAT"/>
+<wire x1="127" y1="-129.54" x2="127" y2="-137.16" width="0.1524" layer="91"/>
+<label x="127" y="-137.16" size="1.778" layer="95"/>
+</segment>
 </net>
 <net name="BUT1" class="0">
@@
 </segment>
 </net>
+<net name="N$21" class="0">
+<segment>
+<pinref part="IC1" gate="G$1" pin="PROG"/>
+<wire x1="99.06" y1="-124.46" x2="88.9" y2="-124.46" width="0.1524" layer="91"/>
+<pinref part="R24" gate="G$1" pin="2"/>
+</segment>
+</net>
+<net name="CHARGE_EN" class="0">
+<segment>
+<pinref part="IC1" gate="G$1" pin="CE"/>
+<wire x1="127" y1="-121.92" x2="139.7" y2="-121.92" width="0.1524" layer="91"/>
+<label x="149.86" y="-121.92" size="1.778" layer="95"/>
+<pinref part="R25" gate="G$1" pin="1"/>
+<wire x1="139.7" y1="-121.92" x2="147.32" y2="-121.92" width="0.1524" layer="91"/>
+<junction x="139.7" y="-121.92"/>
+</segment>
+<segment>
+<pinref part="U$27" gate="G$1" pin="C"/>
+<wire x1="190.5" y1="-121.92" x2="190.5" y2="-119.38" width="0.1524" layer="91"/>
+<label x="190.5" y="-116.84" size="1.778" layer="95"/>
+</segment>
+</net>
+<net name="N$24" class="0">
+<segment>
+<pinref part="IC1" gate="G$1" pin="CHRG"/>
+<wire x1="127" y1="-124.46" x2="129.54" y2="-124.46" width="0.1524" layer="91"/>
+<pinref part="U$15" gate="G$1" pin="C"/>
+</segment>
+</net>
+<net name="N$25" class="0">
+<segment>
+<pinref part="IC1" gate="G$1" pin="STDBY"/>
+<wire x1="127" y1="-127" x2="129.54" y2="-127" width="0.1524" layer="91"/>
+<pinref part="U$26" gate="G$1" pin="C"/>
+</segment>
+</net>
+<net name="N$6" class="0">
+<segment>
+<pinref part="U$26" gate="G$1" pin="A"/>
+<wire x1="137.16" y1="-127" x2="139.7" y2="-127" width="0.1524" layer="91"/>
+<pinref part="R27" gate="G$1" pin="2"/>
+</segment>
+</net>
+<net name="N$16" class="0">
+<segment>
+<pinref part="U$15" gate="G$1" pin="A"/>
+<wire x1="137.16" y1="-124.46" x2="139.7" y2="-124.46" width="0.1524" layer="91"/>
+<pinref part="R26" gate="G$1" pin="2"/>
+</segment>
+</net>
+<net name="N$22" class="0">
+<segment>
+<pinref part="U$27" gate="G$1" pin="B"/>
+<wire x1="182.88" y1="-127" x2="185.42" y2="-127" width="0.1524" layer="91"/>
+<pinref part="R28" gate="G$1" pin="1"/>
+</segment>
+</net>
+<net name="3.3" class="0">
+<segment>
+<pinref part="U$25" gate="G$1" pin="OUT"/>
+<wire x1="88.9" y1="-93.98" x2="91.44" y2="-93.98" width="0.1524" layer="91"/>
+<label x="91.44" y="-93.98" size="1.778" layer="95"/>
+</segment>
+</net>

Commit message: elec v1.1 (wip)
Parts:
- removed JMP: CONNEC_1X02BASIC, rhoban:CONNEC_1X02BASIC
- removed Q1, Q2: BC550C, transistor-npn:BC550C
- added SU-5V: STEPUP-5V, rhoban:STEPUP-5V
- added U$28, U$29: NPN_BC817,215, rhoban:NPN_BC817,215
Connections:
- new net USB+: IC1.VCC, MAPLE.VIN, R25.2
- net GND: now also SU-5V.IN-, SU-5V.OUT-, U$28.E, U$29.E; no longer Q1.E, Q2.E
- net HOLES_GND1: now also U$28.C; no longer Q1.C
- net HOLES_GND2: now also U$29.C; no longer Q2.C
- net N$3: now also U$28.B; no longer Q1.B
- net N$4: now also U$29.B; no longer Q2.B
- net VCC: now also AMP.VIN, R22.2, SU-5V.OUT+; no longer IC1.VCC, JMP.2, MAPLE.VIN, R25.2
- net VIN: now also MAPLE.21, SU-5V.IN+; no longer AMP.VIN, JMP.1, R22.2
Changed lines of the file:
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@@
 <class number="0" name="default" width="0.3048" drill="0">
 </class>
-<class number="1" name="alim" width="0.762" drill="0">
+<class number="1" name="alim" width="0.508" drill="0">
 <clearance class="1" value="0.0762"/>
 </class>
@@
 <part name="R17" library="SparkFun-Passives" deviceset="RESISTOR" device="0805-RES" value="10k"/>
 <part name="R18" library="SparkFun-Passives" deviceset="RESISTOR" device="0805-RES" value="10k"/>
-<part name="JMP" library="rhoban" deviceset="CONNEC_1X02" device="BASIC"/>
 <part name="PWR" library="rhoban" deviceset="CONNEC_1X02" device="BASIC"/>
 <part name="MAPLE" library="rhoban" deviceset="MAPLE_MINI" device=""/>
-<part name="Q1" library="transistor-npn" deviceset="BC550*" device="" technology="C"/>
-<part name="Q2" library="transistor-npn" deviceset="BC550*" device="" technology="C"/>
 <part name="R1" library="SparkFun-Passives" deviceset="RESISTOR" device="0805-RES" value="1k"/>
 <part name="R2" library="SparkFun-Passives" deviceset="RESISTOR" device="0805-RES" value="1k"/>
@@
 <part name="U$27" library="rhoban" deviceset="NPN" device="_BC817,215"/>
 <part name="R28" library="SparkFun-Passives" deviceset="RESISTOR" device="0805-RES" value="2K"/>
+<part name="SU-5V" library="rhoban" deviceset="STEPUP-5V" device=""/>
+<part name="U$28" library="rhoban" deviceset="NPN" device="_BC817,215"/>
+<part name="U$29" library="rhoban" deviceset="NPN" device="_BC817,215"/>
 </parts>
 <sheets>
@@
 <instance part="R17" gate="G$1" x="223.52" y="-15.24" rot="R270"/>
 <instance part="R18" gate="G$1" x="226.06" y="-58.42" rot="R270"/>
-<instance part="JMP" gate="G$1" x="83.82" y="-43.18"/>
 <instance part="PWR" gate="G$1" x="83.82" y="-58.42"/>
 <instance part="MAPLE" gate="G$1" x="78.74" y="35.56"/>
-<instance part="Q1" gate="G$1" x="226.06" y="-104.14"/>
-<instance part="Q2" gate="G$1" x="261.62" y="-104.14"/>
 <instance part="R1" gate="G$1" x="215.9" y="-104.14"/>
 <instance part="R2" gate="G$1" x="251.46" y="-104.14"/>
@@
 <instance part="U$27" gate="G$1" x="187.96" y="-127"/>
 <instance part="R28" gate="G$1" x="177.8" y="-127" rot="R180"/>
+<instance part="SU-5V" gate="G$1" x="60.96" y="-152.4"/>
+<instance part="U$28" gate="G$1" x="226.06" y="-104.14"/>
+<instance part="U$29" gate="G$1" x="261.62" y="-104.14"/>
 </instances>
 <busses>
@@
 </segment>
 <segment>
-<pinref part="Q1" gate="G$1" pin="E"/>
 <wire x1="228.6" y1="-109.22" x2="228.6" y2="-114.3" width="0.1524" layer="91"/>
 <wire x1="228.6" y1="-114.3" x2="241.3" y2="-114.3" width="0.1524" layer="91"/>
 <wire x1="241.3" y1="-121.92" x2="241.3" y2="-114.3" width="0.1524" layer="91"/>
-<pinref part="Q2" gate="G$1" pin="E"/>
 <wire x1="241.3" y1="-114.3" x2="264.16" y2="-114.3" width="0.1524" layer="91"/>
 <wire x1="264.16" y1="-114.3" x2="264.16" y2="-109.22" width="0.1524" layer="91"/>
 <label x="238.76" y="-124.46" size="1.778" layer="95"/>
+<pinref part="U$28" gate="G$1" pin="E"/>
+<pinref part="U$29" gate="G$1" pin="E"/>
 </segment>
 <segment>
@@
 <label x="190.5" y="-137.16" size="1.778" layer="95"/>
 </segment>
-</net>
-<net name="VCC" class="0">
-<segment>
-<pinref part="JMP" gate="G$1" pin="2"/>
-<wire x1="86.36" y1="-43.18" x2="78.74" y2="-43.18" width="0.1524" layer="91"/>
-<label x="71.12" y="-43.18" size="1.778" layer="95"/>
-</segment>
-<segment>
-<pinref part="MAPLE" gate="G$1" pin="VIN"/>
-<wire x1="96.52" y1="-12.7" x2="101.6" y2="-12.7" width="0.1524" layer="91"/>
-<label x="104.14" y="-12.7" size="1.778" layer="95"/>
-</segment>
+<segment>
+<pinref part="SU-5V" gate="G$1" pin="IN-"/>
+<wire x1="55.88" y1="-142.24" x2="53.34" y2="-142.24" width="0.1524" layer="91"/>
+<label x="48.26" y="-142.24" size="1.778" layer="95"/>
+</segment>
+<segment>
+<pinref part="SU-5V" gate="G$1" pin="OUT-"/>
+<wire x1="83.82" y1="-142.24" x2="86.36" y2="-142.24" width="0.1524" layer="91"/>
+<label x="86.36" y="-142.24" size="1.778" layer="95"/>
+</segment>
+</net>
+<net name="VCC" class="1">
 <segment>
 <wire x1="132.08" y1="-20.32" x2="129.54" y2="-20.32" width="0.1524" layer="91"/>
@@
 </segment>
 <segment>
-<pinref part="IC1" gate="G$1" pin="VCC"/>
-<wire x1="99.06" y1="-129.54" x2="96.52" y2="-129.54" width="0.1524" layer="91"/>
-<label x="88.9" y="-129.54" size="1.778" layer="95"/>
-</segment>
-<segment>
-<pinref part="R25" gate="G$1" pin="2"/>
-<wire x1="139.7" y1="-111.76" x2="139.7" y2="-109.22" width="0.1524" layer="91"/>
-<label x="139.7" y="-109.22" size="1.778" layer="95"/>
-</segment>
-<segment>
 <pinref part="R26" gate="G$1" pin="1"/>
 <wire x1="149.86" y1="-124.46" x2="152.4" y2="-124.46" width="0.1524" layer="91"/>
@@
 <wire x1="149.86" y1="-127" x2="152.4" y2="-127" width="0.1524" layer="91"/>
 <label x="152.4" y="-127" size="1.778" layer="95"/>
+</segment>
+<segment>
+<pinref part="SU-5V" gate="G$1" pin="OUT+"/>
+<wire x1="83.82" y1="-149.86" x2="86.36" y2="-149.86" width="0.1524" layer="91"/>
+<label x="86.36" y="-149.86" size="1.778" layer="95"/>
+</segment>
+<segment>
+<pinref part="AMP" gate="G$1" pin="VIN"/>
+<wire x1="289.56" y1="17.78" x2="287.02" y2="17.78" width="0.1524" layer="91"/>
+<label x="281.94" y="17.78" size="1.778" layer="95"/>
+</segment>
+<segment>
+<pinref part="R22" gate="G$1" pin="2"/>
+<wire x1="284.48" y1="38.1" x2="284.48" y2="40.64" width="0.1524" layer="91"/>
+<label x="284.48" y="40.64" size="1.778" layer="95" rot="R90"/>
 </segment>
 </net>
@@
 <net name="VIN" class="1">
 <segment>
-<pinref part="JMP" gate="G$1" pin="1"/>
-<wire x1="86.36" y1="-40.64" x2="78.74" y2="-40.64" width="0.1524" layer="91"/>
-<label x="71.12" y="-40.64" size="1.778" layer="95"/>
-</segment>
-<segment>
-<pinref part="AMP" gate="G$1" pin="VIN"/>
-<wire x1="289.56" y1="17.78" x2="287.02" y2="17.78" width="0.1524" layer="91"/>
-<label x="281.94" y="17.78" size="1.778" layer="95"/>
-</segment>
-<segment>
 <pinref part="U$14" gate="G$1" pin="+"/>
 <wire x1="30.48" y1="-33.02" x2="30.48" y2="-30.48" width="0.1524" layer="91"/>
@@
 </segment>
 <segment>
-<pinref part="R22" gate="G$1" pin="2"/>
-<wire x1="284.48" y1="38.1" x2="284.48" y2="40.64" width="0.1524" layer="91"/>
-<label x="284.48" y="40.64" size="1.778" layer="95" rot="R90"/>
-</segment>
-<segment>
 <wire x1="335.28" y1="-7.62" x2="335.28" y2="-12.7" width="0.1524" layer="91"/>
 <pinref part="R14" gate="G$1" pin="1"/>
@@
 <pinref part="R28" gate="G$1" pin="2"/>
 </segment>
+<segment>
+<pinref part="SU-5V" gate="G$1" pin="IN+"/>
+<wire x1="55.88" y1="-149.86" x2="53.34" y2="-149.86" width="0.1524" layer="91"/>
+<label x="48.26" y="-149.86" size="1.778" layer="95"/>
+</segment>
+<segment>
+<pinref part="MAPLE" gate="G$1" pin="21"/>
+<wire x1="71.12" y1="12.7" x2="68.58" y2="12.7" width="0.1524" layer="91"/>
+<label x="60.96" y="12.7" size="1.778" layer="95"/>
+</segment>
 </net>
 <net name="AUDIO" class="0">
@@
 </segment>
 <segment>
-<pinref part="Q1" gate="G$1" pin="C"/>
 <wire x1="228.6" y1="-99.06" x2="228.6" y2="-96.52" width="0.1524" layer="91"/>
 <label x="228.6" y="-96.52" size="1.778" layer="95"/>
+<pinref part="U$28" gate="G$1" pin="C"/>
 </segment>
 </net>
@@
 </segment>
 <segment>
-<pinref part="Q2" gate="G$1" pin="C"/>
 <wire x1="264.16" y1="-99.06" x2="264.16" y2="-96.52" width="0.1524" layer="91"/>
 <label x="264.16" y="-96.52" size="1.778" layer="95"/>
+<pinref part="U$29" gate="G$1" pin="C"/>
 </segment>
 </net>
@@
 <segment>
 <pinref part="R1" gate="G$1" pin="2"/>
-<pinref part="Q1" gate="G$1" pin="B"/>
 <wire x1="220.98" y1="-104.14" x2="223.52" y2="-104.14" width="0.1524" layer="91"/>
+<pinref part="U$28" gate="G$1" pin="B"/>
 </segment>
 </net>
@@
 <segment>
 <pinref part="R2" gate="G$1" pin="2"/>
-<pinref part="Q2" gate="G$1" pin="B"/>
 <wire x1="256.54" y1="-104.14" x2="259.08" y2="-104.14" width="0.1524" layer="91"/>
+<pinref part="U$29" gate="G$1" pin="B"/>
 </segment>
 </net>
@@
 </segment>
 </net>
+<net name="USB+" class="0">
+<segment>
+<pinref part="MAPLE" gate="G$1" pin="VIN"/>
+<wire x1="96.52" y1="-12.7" x2="101.6" y2="-12.7" width="0.1524" layer="91"/>
+<label x="104.14" y="-12.7" size="1.778" layer="95"/>
+</segment>
+<segment>
+<pinref part="IC1" gate="G$1" pin="VCC"/>
+<wire x1="99.06" y1="-129.54" x2="96.52" y2="-129.54" width="0.1524" layer="91"/>
+<label x="88.9" y="-129.54" size="1.778" layer="95"/>
+</segment>
+<segment>
+<pinref part="R25" gate="G$1" pin="2"/>
+<wire x1="139.7" y1="-111.76" x2="139.7" y2="-109.22" width="0.1524" layer="91"/>
+<label x="139.7" y="-109.22" size="1.778" layer="95"/>
+</segment>
+</net>
