File: electronics/v1.2s/flute.brd (EAGLE design)
At the start: 25 x 250 mm, 96 parts, among them IC1 TP4056, IC2 MCP1703T-3302E/CB, IC3 MCP1703T-3302E/CB, P1 PRESSURE_SENSOR, U1 CD4051BM, U2 CD4051BM, U3 SSM2211SZ, X1 USB-MINIB

Commit message: Version simplified
Parts:
- removed BTN: CONNEC_1X02BASIC, rhoban:CONNEC_1X02
- removed C13: 18pF, SparkFun:C0402
- removed C5: 1uF, SparkFun:C0402
- removed R29: 0.4, SparkFun-Passives:0805
- added C18: 10uF, SparkFun-Passives:0805
- added C20, C21: 18pF, SparkFun-Passives:0805
- added U$16: SWITCHKCD11, rhoban:KCD11
- C10, C11, C6, C7, C8: device SparkFun:C0402 -> SparkFun-Passives:0805
- C12: value 18pF -> 1uF; device SparkFun:C0402 -> SparkFun-Passives:0805
- moved C7 50.0 mm to (2.20, 89.2)
- moved C8 50.0 mm to (22.4, 90.9), turned to 0 degrees
- moved C6 47.0 mm to (2.20, 90.8)
- moved U$9 31.7 mm to (3.55, 65.2)
- moved PWR 12.6 mm to (2.56, 45.7)
- moved C12 9.89 mm to (2.20, 92.4)
- moved C10 5.87 mm to (4.00, 41.8), turned to 180 degrees
- moved C11 5.76 mm to (7.30, 41.9)
- moved R31 5.44 mm to (4.00, 39.9), turned to 180 degrees
- moved R32 5.14 mm to (7.20, 40.0), turned to 0 degrees
- moved R28 3.85 mm to (7.40, 44.0)
- moved C14 2.83 mm to (14.0, 43.6)
- moved R33 2.75 mm to (9.95, 42.1), turned to 270 degrees
- moved R24 1.75 mm to (20.6, 62.0)
- moved PROGRAM 1.66 mm to (23.2, 94.8)
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Connections:
- removed net N$23: C2.2, IC1.4, R29.2
- net 33: now also C12.2, C6.2, C7.2; no longer C6.1, C7.1, C8.1
- net AV+: now also C8.1; no longer C5.1
- net GND: now also C12.1, C18.1, C20.1, C21.1, C6.1, C7.1; no longer C12.2, C13.2, C5.2, C6.2, C7.2
- net OSC_IN: now also C21.2; no longer C12.1
- net OSC_OUT: now also C20.2; no longer C13.1
- net USB+: now also C2.2, IC1.4; no longer R29.1
- net VIN: now also C18.2, U$16.B1, U$16.B2; no longer BTN.2
- net VIN_BAT: now also U$16.A1, U$16.A2; no longer BTN.1
Routing:
- net RX1: track 54.8 -> 13.0 mm, vias 5 -> 3
- net BRX: track 124.3 -> 162.8 mm, vias 6 -> 2
- net HOLE7: track 108.6 -> 142.7 mm
- net HOLES_GND1: track 176.6 -> 148.6 mm, vias 3 -> 7
- net GND: track 590.9 -> 564.1 mm, vias 14 -> 12
- net HOLES_GND2: track 140.8 -> 166.7 mm, vias 1 -> 2
- net BTX: track 151.6 -> 126.3 mm
- net AUDIO: track 66.9 -> 43.8 mm, vias 2 -> 4
- net 33: track 272.8 -> 293.6 mm
- net N$29: track 61.6 -> 42.2 mm, vias 4 -> 2
- net OSC_IN: track 28.0 -> 47.2 mm, vias 4 -> 0
- net VIN_BAT: track 28.0 -> 44.8 mm, vias 1 -> 2
- net HOLES_EN1: track 46.6 -> 30.9 mm, vias 4 -> 2
- net HOLE1: track 73.5 -> 58.2 mm
- net VIN: track 262.9 -> 248.1 mm
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Other:
- board text added: "GND"
