File: electronics/v1.2s/flute.sch (EAGLE design)
At the start: 96 parts, among them IC1 TP4056, IC2 MCP1703T-3302E/CB, IC3 MCP1703T-3302E/CB, P1 PRESSURE_SENSOR, U1 CD4051BM, U2 CD4051BM, U3 SSM2211SZ, X1 USB-MINIB

Commit message: Version simplified
Parts:
- removed BTN: CONNEC_1X02BASIC, rhoban:CONNEC_1X02BASIC
- removed C13: 18pF, SparkFun:CAP0402
- removed C5: 1uF, SparkFun:CAP0402
- removed R29: 0.4, SparkFun-Passives:RESISTOR0805-RES
- added C18: 10uF, SparkFun-Passives:CAP0805
- added C20, C21: 18pF, SparkFun-Passives:CAP0805
- added U$16: SWITCHKCD11, rhoban:SWITCHKCD11
- C10, C11, C6, C7, C8: device SparkFun:CAP0402 -> SparkFun-Passives:CAP0805
- C12: value 18pF -> 1uF; device SparkFun:CAP0402 -> SparkFun-Passives:CAP0805
Connections:
- removed net N$23: C2.2, IC1.VCC, R29.2
- net 33: now also C12.2, C6.2, C7.2; no longer C6.1, C7.1, C8.1
- net AV+: now also C8.1; no longer C5.1
- net GND: now also C12.1, C18.1, C20.1, C21.1, C6.1, C7.1; no longer C12.2, C13.2, C5.2, C6.2, C7.2
- net OSC_IN: now also C21.2; no longer C12.1
- net OSC_OUT: now also C20.2; no longer C13.1
- net USB+: now also C2.2, IC1.VCC; no longer R29.1
- net VIN: now also C18.2, U$16.P$2; no longer BTN.2
- net VIN_BAT: now also U$16.P$1; no longer BTN.1
Other:
- moved on the sheet: C12, C6, C7, C8
